File: tigard.kicad_pcb (KiCad board)
At the start: 4 copper layers, 46 x 46 mm, 92 parts, among them J1 USB_C_Receptacle_USB2.0, J2 JTAG, J3 UART, J4 SPI, J5 CORTEX, J6 LA, J7 I2C, Q1 BSH103, SW1 TARGET, SW2 MODE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

Commit message: Add fidutials
Parts:
- added FID1: Fiducial, Fiducial:Fiducial_0.5mm_Mask1mm, F.Cu at (31.6, 35.9)
- added FID2: Fiducial, Fiducial:Fiducial_0.5mm_Mask1mm, F.Cu at (31.8, 70.2)
- added FID3: Fiducial, Fiducial:Fiducial_0.5mm_Mask1mm, F.Cu at (69.5, 33.5)
Connections:
- J1 pad A8: (no net) -> Net-(J1-PadA8)
- J1 pad B8: (no net) -> Net-(J1-PadB8)
- J5 pad 7: (no net) -> Net-(J5-Pad7)
- J6 pad 11: (no net) -> Net-(J6-Pad11)
- J6 pad 12: (no net) -> Net-(J6-Pad12)
- J6 pad 13: (no net) -> Net-(J6-Pad13)
- J6 pad 14: (no net) -> Net-(J6-Pad14)
- RN6 pad 3: (no net) -> Net-(RN6-Pad3)
- RN6 pad 4: (no net) -> Net-(RN6-Pad4)
- SW1 pad 1: (no net) -> Net-(SW1-Pad1)
- SW1 pad 2: (no net) -> Net-(SW1-Pad2)
- SW1 pad 3: (no net) -> Net-(SW1-Pad3)
- SW1 pad 4: (no net) -> Net-(SW1-Pad4)
- SW1 pad 5: (no net) -> Net-(SW1-Pad5)
- U1 pad 4: (no net) -> Net-(U1-Pad4)
- U2 pad 4: (no net) -> Net-(U2-Pad4)
- U3 pad 24: (no net) -> Net-(U3-Pad24)
- U3 pad 26: (no net) -> Net-(U3-Pad26)
- U3 pad 27: (no net) -> Net-(U3-Pad27)
- U3 pad 28: (no net) -> Net-(U3-Pad28)
- U3 pad 32: (no net) -> Net-(U3-Pad32)
- U3 pad 33: (no net) -> Net-(U3-Pad33)
- U3 pad 34: (no net) -> Net-(U3-Pad34)
- U3 pad 36: (no net) -> Net-(U3-Pad36)
- U3 pad 48: (no net) -> Net-(U3-Pad48)
- U3 pad 52: (no net) -> Net-(U3-Pad52)
- U3 pad 53: (no net) -> Net-(U3-Pad53)
- U3 pad 54: (no net) -> Net-(U3-Pad54)
- U3 pad 55: (no net) -> Net-(U3-Pad55)
- U3 pad 57: (no net) -> Net-(U3-Pad57)
- U3 pad 58: (no net) -> Net-(U3-Pad58)
- U3 pad 59: (no net) -> Net-(U3-Pad59)

Commit message: Set soldermask clerance to zero
Other:
- rule pad_to_mask_clearance: 0.05 -> 0
Changed lines of the file:
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@@
     (pad_size 2 2)
     (pad_drill 1)
-    (pad_to_mask_clearance 0.05)
+    (pad_to_mask_clearance 0)
     (aux_axis_origin 76 76)
     (grid_origin 1 -0.05)
